Commit message: rviz

File: src/rob2w_description/src/urdf/rob2w.xacro (robot description, xacro)
@@ -69,64 +69,28 @@
         <cylinder length = "0.02" radius = "0.015" />
       </geometry>
-      <material name="blue"/>
+      <color rgba="0.0 0.0 0.58515625 0.5"/>
     </visual>
-  </link>
   <!-- Create wheel right -->
-  <link name="link_right_wheel">
-    <inertial>
-      <mass value="0.02"/>
-      <origin rpy="0 1.5707 1.5707" xyz="0 0 0"/>
-      <inertia ixx="0.00052666666" ixy="0" ixz="0" iyy="0.00052666666" iyz="0" izz="0.001"/>
-    </inertial>
-    <collision name="link_right_wheel_collision">
-      <origin rpy="0 1.5707 1.5707" xyz="0 0 0" />
+    <visual name="link_right_wheel_visual">
+      <origin rpy="0 1.5707 1.5707" xyz="0 0.02 0"/>
       <geometry>
         <cylinder length="0.004" radius="0.01"/>
       </geometry>
-    </collision>
-    <visual name="link_right_wheel_visual">
-      <origin rpy="0 1.5707 1.5707" xyz="0 0 0"/>
+      <color rgba="0.80078125 0.12890625 0.1328125 1.0"/>
+    </visual>
+    <visual name="link_left_wheel_visual">
+      <origin rpy="0 1.5707 1.5707" xyz="0 -0.02 0"/>
       <geometry>
         <cylinder length="0.004" radius="0.01"/>
       </geometry>
+      <color rgba="0.80078125 0.12890625 0.1328125 1.0"/>
+    </visual>
+    <visual name="arrow_visual">
+      <origin rpy="0 1.5707 1.5707" xyz="0.02 0 0.01"/>
+      <geometry>
+        <box size="0.01 0.01 0.005"/>
+      </geometry>
+      <color rgba="0.0 0.8 0.0 1.0"/>
     </visual>
   </link>
-  <!--   Joint for right wheel  -->
-  <joint name="joint_right_wheel" type="continuous">
-    <origin rpy="0 0 0" xyz="0.0 0.02 0"/>
-    <child link="link_right_wheel" />
-    <parent link="base_link"/>
-    <axis rpy="0 0 0" xyz="0 1 0"/>
-    <limit effort="10000" velocity="1000"/>
-    <joint_properties damping="1.0" friction="1.0" />
-  </joint>
-  <!-- Left Wheel link -->
-  <link name="link_left_wheel">
-    <inertial>
-      <mass value="0.02"/>
-      <origin rpy="0 1.5707 1.5707" xyz="0 0 0"/>
-      <inertia ixx="0.00052666666" ixy="0" ixz="0" iyy="0.00052666666" iyz="0" izz="0.001"/>
-    </inertial>
-    <collision name="link_left_wheel_collision">
-      <origin rpy="0 1.5707 1.5707" xyz="0 0 0" />
-      <geometry>
-        <cylinder length="0.004" radius="0.01"/>
-      </geometry>
-    </collision>
-    <visual name="link_left_wheel_visual">
-      <origin rpy="0 1.5707 1.5707" xyz="0 0 0"/>
-      <geometry>
-        <cylinder length="0.004" radius="0.01"/>
-      </geometry>
-    </visual>
-  </link>
-  <!--   Joint for right wheel  -->
-  <joint name="joint_left_wheel" type="continuous">
-    <origin rpy="0 0 0" xyz="0 -0.02 0"/>
-    <child link="link_left_wheel" />
-    <parent link="base_link"/>
-    <axis rpy="0 0 0" xyz="0 1 0"/>
-    <limit effort="10000" velocity="1000"/>
-    <joint_properties damping="1.0" friction="1.0" />
-  </joint>
 </robot>

Commit message: rviz turtle and simul

File: src/rob2w_description/src/urdf/rob2w.xacro (robot description, xacro)
@@ -28,5 +28,5 @@
     <color rgba="1.0 1.0 1.0 1.0"/>
   </material>
-  <gazebo reference="base_link">
+  <gazebo reference="base_link_rob2w">
     <material>Gazebo/Orange</material>
   </gazebo>
@@ -37,5 +37,5 @@
     <material>Gazebo/Blue</material>
   </gazebo>
-  <link name="base_link">
+  <link name="base_link_rob2w">
     <!-- pose and inertial -->
     <pose>0 0 0.1 0 0 0</pose>
